Commit message: feat(sim): weld cubes to the gripper with DetachableJoint
Adds three gz-sim-detachable-joint-system plugins to the robot
description (one per cube colour, since child_model is fixed at load
time) and bridges the six /grasp/<colour>/{attach,detach} std_msgs/Empty
topics ROS_TO_GZ. parent_link is link5, not end_effector_link: gripper_joint
and end_effector_joint are both fixed, so sdformat lumps gripper_link and
end_effector_link into link5, and the other names don't exist as Gazebo
links. The grasp_joint xacro macro is defined at the robot root next to
position_joint/mimic_joint, not nested inside <gazebo>, so a failure to
expand isn't silent.

Verified against a live launch of pick_place.launch.py (see
task-4-report.md for full detail and exact poses):
- The cube is NOT welded when it merely appears: 5 s after spawn it sits
  at its spawn pose on the pedestal, and publishing detach with nothing
  attached is a no-op that leaves it untouched. Task 6's detach-on-startup
  is therefore not required for this failure mode, though it remains
  harmless as a safety net.
- Attach does NOT teleport the cube: with the arm parked at link5 far from
  the cube, the cube's pose is bit-for-bit identical before and after
  publishing attach.
- The weld holds through motion: after attach, driving the arm via
  /arm_controller/joint_trajectory moved the cube along with link5, and
  publishing detach dropped it to the floor.

Also fixes the sim_gait.py file mode. It was tracked as 100644; with
--symlink-install, install(PROGRAMS ...) symlinks to the source file, so
the non-executable bit survives and ros2 launch fails to run it on a
fresh checkout. That would have blocked verification of this task, so
the fix is bundled here.

Co-Authored-By: Claude Opus 5 <noreply@anthropic.com>

File: ROSpider/src/simulations/rospider_gazebo/urdf/rospider_gazebo.urdf.xacro (robot description, xacro)
@@ -53,4 +53,21 @@
     </joint>
   </xacro:macro>
+  <!-- Grasping is a joint attachment, not friction: the gripper is small, has
+       five mimic fingers and would drop a 5 cm cube. parent_link must be link5
+       because gripper_joint and end_effector_joint are fixed, so sdformat lumps
+       gripper_link and end_effector_link into link5. child_model is fixed at
+       load time, hence one plugin per cube. suppress_child_warning is needed
+       because pick_place.launch.py spawns the cubes after the robot. -->
+  <xacro:macro name="grasp_joint" params="colour">
+    <plugin filename="gz-sim-detachable-joint-system"
+            name="gz::sim::systems::DetachableJoint">
+      <parent_link>link5</parent_link>
+      <child_model>pick_cube_${colour}</child_model>
+      <child_link>link</child_link>
+      <attach_topic>/grasp/${colour}/attach</attach_topic>
+      <detach_topic>/grasp/${colour}/detach</detach_topic>
+      <suppress_child_warning>true</suppress_child_warning>
+    </plugin>
+  </xacro:macro>
   <ros2_control name="GazeboSimSystem" type="system">
     <hardware>
@@ -93,4 +110,7 @@
       <dimensions>2</dimensions>
     </plugin>
+    <xacro:grasp_joint colour="red"/>
+    <xacro:grasp_joint colour="green"/>
+    <xacro:grasp_joint colour="blue"/>
   </gazebo>
   <!-- LD19-like 2D LiDAR. min range 0.2 m matches the real robot's laser filter
